File: mesa_aquecida/hardware/hardware.kicad_pcb (KiCad board)
At the start: 2 copper layers, 35 parts, among them J1 Conn_01x04_Male, J10 Conn_01x04_Male, J2 Conn_01x04_Male, J3 Conn_01x04_Male, J4 Conn_01x02_Female, J5 Conn_01x02_Male, J6 Conn_01x02_Male, J7 Conn_01x02_Male, J8 Conn_01x02_Male, J9 Screw_Terminal_01x03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

Commit message: Created pcb
Parts:
- added H1: MountingHole, MountingHole:MountingHole_4.3mm_M4, F.Cu at (178.8, 95.0)
- added H2: MountingHole, MountingHole:MountingHole_4.3mm_M4, F.Cu at (220.0, 79.8)
- added H3: MountingHole, MountingHole:MountingHole_4.3mm_M4, F.Cu at (183.4, 79.8)
- added H4: MountingHole, MountingHole:MountingHole_4.3mm_M4, F.Cu at (220.5, 94.5)
- added J11: Screw_Terminal_01x02, TerminalBlock:TerminalBlock_bornier-2_P5.08mm, F.Cu at (219.5, 31.0)
- added J12: Conn_01x02_Female, Connector_PinHeader_2.54mm:PinHeader_1x02_P2.54mm_Vertical, F.Cu at (193.5, 79.8)
- J2: value Conn_01x04_Male -> Conn_01x02_Female; footprint Connector_PinHeader_2.54mm:PinHeader_1x04_P2.54mm_Vertical -> Connector_PinHeader_2.54mm:PinHeader_1x02_P2.54mm_Vertical
- moved J2 32.8 mm to (178.8, 47.8), turned to 180 degrees
- moved SW1 25.1 mm to (214.9, 95.0), turned to 180 degrees
- moved SW3 20.6 mm to (195.6, 95.0), turned to 180 degrees
- moved D3 20.6 mm to (210.8, 36.6), turned to 0 degrees
- moved R2 19.8 mm to (190.0, 61.5), turned to 270 degrees
- moved R4 15.9 mm to (187.5, 61.5), turned to 270 degrees
- moved R6 12.1 mm to (184.9, 61.5), turned to 270 degrees
- moved R8 11.5 mm to (185.4, 34.6)
- moved Q1 11.2 mm to (189.5, 37.1), turned to 270 degrees
- moved R1 8.63 mm to (199.1, 69.1), turned to 180 degrees
- moved C1 8.19 mm to (203.7, 69.1)
- moved C2 8.12 mm to (204.2, 62.0)
- moved C4 7.18 mm to (214.4, 71.6), turned to 0 degrees
- moved C3 7.11 mm to (214.4, 68.6), turned to 0 degrees
- moved R9 4.06 mm to (194.1, 39.6)
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Connections:
- J2 pad 1: +5V -> GND
- J2 pad 2: GND -> +5V
- J9 pad 2: Net-(D3-Pad1) -> Net-(J9-Pad2)
- R3 pad 2: SDA -> SCL
- R5 pad 2: SCL -> SDA
- U1 pad 13: POWER -> Net-(U1-Pad13)
- U1 pad 2: Net-(U1-Pad2) -> NTC
- U1 pad 5: NTC -> POWER
Routing:
- net +3V3: track 0.00 -> 139.2 mm
- net GND: track 0.00 -> 64.2 mm, vias 0 -> 2
- net +12V: track 0.00 -> 42.7 mm
- net POWER: track 0.00 -> 38.8 mm
- net Net-(J10-Pad1): track 0.00 -> 38.2 mm
- net Net-(D3-Pad1): track 0.00 -> 31.7 mm
- net GND1: track 0.00 -> 30.5 mm
- net NTC: track 0.00 -> 23.5 mm
- net Net-(J10-Pad2): track 0.00 -> 23.1 mm
- net Net-(J1-Pad1): track 0.00 -> 19.2 mm
- net +5V: track 0.00 -> 19.1 mm
- net RST: track 0.00 -> 18.2 mm
- net Net-(J1-Pad2): track 0.00 -> 14.4 mm
- net Net-(J10-Pad3): track 0.00 -> 12.8 mm
- net Net-(Q1-Pad3): track 0.00 -> 12.4 mm
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- added copper zone on B.Cu, net GND
Other:
- board outline added: 49.3 x 80.8 mm
- net class Default: clearance 0.2 -> 0.3048; trace_width 0.25 -> 0.762; via_dia 0.8 -> 1.8; via_drill 0.4 -> 1
- net class Power added: clearance 0.3048, trace_width 2.5, via_dia 1.8, via_drill 1
- rule trace_clearance: 0.2 -> 0.3048
- board text added: "Display comm."
- board text added: "Display power"
- board text removed: "Display"

Commit message: Added aligment hole
Parts:
- moved C6 51.5 mm to (172.2, 96.0)
- moved J1 51.5 mm to (138.2, 104.6)
- moved SW3 51.5 mm to (154.4, 126.0)
- moved J10 51.5 mm to (143.3, 129.0)
- moved J6 51.5 mm to (163.1, 82.3)
- moved J8 51.5 mm to (143.8, 82.3)
- moved C1 51.5 mm to (162.6, 100.1)
- moved C2 51.5 mm to (163.0, 93.0)
- moved C3 51.5 mm to (173.2, 99.6)
- moved C4 51.5 mm to (173.2, 102.6)
- moved C5 51.5 mm to (174.8, 96.0)
- moved D1 51.5 mm to (173.2, 108.6)
- moved D3 51.5 mm to (169.7, 67.6)
- moved H1 51.5 mm to (137.7, 126.0)
- moved H2 51.5 mm to (178.8, 110.7)
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Routing:
- net Net-(J10-Pad1): track 38.2 -> 33.6 mm
- net (no net): vias 0 -> 1

Commit message: Adicionado corte
Routing:
- added copper zone on B.Cu, net GND1
Other:
- outline, holes or cut-outs redrawn
Changed lines of the file:
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@@
   (general
     (thickness 1.6)
-    (drawings 12)
+    (drawings 18)
     (tracks 181)
     (zones 0)
@@
     )
   )
+  (gr_line (start 133.604 51.308) (end 133.604 117.348) (layer Edge.Cuts) (width 0.05))
+  (gr_line (start 182.88 117.348) (end 182.88 51.308) (layer Edge.Cuts) (width 0.05))
+  (gr_line (start 133.604 117.348) (end 182.88 117.348) (layer Edge.Cuts) (width 0.05))
+  (gr_line (start 133.604 117.856) (end 134.112 117.856) (layer Edge.Cuts) (width 0.05))
+  (gr_line (start 133.604 132.08) (end 133.604 117.856) (layer Edge.Cuts) (width 0.05))
+  (gr_line (start 182.88 117.856) (end 182.372 117.856) (layer Edge.Cuts) (width 0.05))
+  (gr_line (start 182.88 132.08) (end 182.88 117.856) (layer Edge.Cuts) (width 0.05))
+  (gr_line (start 134.112 117.856) (end 182.372 117.856) (layer Edge.Cuts) (width 0.05))
   (dimension 80.772 (width 0.15) (layer Dwgs.User)
     (gr_text "80.772 mm" (at 191.292 91.694 90) (layer Dwgs.User)
@@
     (effects (font (size 1 1) (thickness 0.15)))
   )
-  (gr_line (start 133.604 132.08) (end 133.604 51.308) (layer Edge.Cuts) (width 0.05))
   (gr_line (start 182.88 132.08) (end 133.604 132.08) (layer Edge.Cuts) (width 0.05))
-  (gr_line (start 182.88 51.308) (end 182.88 132.08) (layer Edge.Cuts) (width 0.05))
   (gr_line (start 133.604 51.308) (end 182.88 51.308) (layer Edge.Cuts) (width 0.05))
   (gr_text "Mini buck : 12V to 5V" (at 153.416 78.232) (layer F.SilkS)
@@
     (polygon
       (pts
-        (xy 131.572 48.768) (xy 187.452 48.768) (xy 185.42 138.176) (xy 128.524 137.16) (xy 129.54 48.768)
-        (xy 131.064 48.26)
+        (xy 132.588 50.292) (xy 184.912 50.292) (xy 185.42 117.348) (xy 132.588 117.348)
       )
     )
+  )
+  (zone (net 25) (net_name GND1) (layer B.Cu) (hatch edge 0.508)
+    (connect_pads (clearance 0.508))
+    (min_thickness 0.254)
+    (fill yes (arc_segments 32) (thermal_gap 0.508) (thermal_bridge_width 0.508))
+    (polygon
+      (pts
+        (xy 184.404 133.096) (xy 133.096 133.096) (xy 133.096 117.856) (xy 184.404 117.856)
+      )
+    )

Commit message: Updated software
Parts:
- C1: value 100n -> 1n
- R7: value 62k -> 82k
- moved R8 23.9 mm to (151.4, 88.4), turned to 0 degrees
Connections:
- R8 pad 1: POWER -> +3V3
- R8 pad 2: GND -> POWER
Routing:
- net +3V3: track 139.2 -> 143.2 mm
- net GND: track 64.2 -> 62.7 mm
- net POWER: track 38.8 -> 38.1 mm
